File: BSidesDFW_2018_Badge.sch (KiCad schematic (older format))
At the start: 6 parts, among them J1 RJ45, J2 RJ45, J3 RJ45, J4 RJ45

Commit message: getting-shit-done
Parts:
- C1, C2: footprint (none) -> BSidesDFW_2018_Badge:C_Rect_L4.6mm_W2.0mm_P2.50mm_MKS02_FKP02
- J1, J2, J3, J4: footprint (none) -> BSidesDFW_2018_Badge:RJHSE538X
Connections:
- net SIG4: now also C1.1
- net SIG5: now also C1.2
- net SIG7: now also C2.1
- net SIG8: now also C2.2
Changed lines of the file:
@@
 EESchema Schematic File Version 2
-LIBS:power
-LIBS:device
-LIBS:transistors
-LIBS:conn
-LIBS:linear
-LIBS:regul
-LIBS:74xx
-LIBS:cmos4000
-LIBS:adc-dac
-LIBS:memory
-LIBS:xilinx
-LIBS:special
-LIBS:microcontrollers
-LIBS:dsp
-LIBS:microchip
-LIBS:analog_switches
-LIBS:motorola
-LIBS:texas
-LIBS:intel
-LIBS:audio
-LIBS:interface
-LIBS:digital-audio
-LIBS:philips
-LIBS:display
-LIBS:cypress
-LIBS:siliconi
-LIBS:opto
-LIBS:atmel
-LIBS:contrib
-LIBS:valves
+LIBS:BSidesDFW_2018_Badge
+LIBS:BSidesDFW_2018_Badge-cache
 EELAYER 25 0
 EELAYER END
@@
 NoConn ~ 5250 4500
 NoConn ~ 5150 4500
-Wire Wire Line
-	4650 2300 4650 2400
-Wire Wire Line
-	5850 5300 5850 5400
-Connection ~ 6150 4100
-Wire Wire Line
-	6150 4500 6150 3800
-Wire Wire Line
-	7250 3800 4350 3800
-Connection ~ 6150 3800
-Connection ~ 4550 4100
-Wire Wire Line
-	4850 4500 4850 4400
-Wire Wire Line
-	4850 4400 4550 4400
-Wire Wire Line
-	4550 4400 4550 3600
-Connection ~ 6250 3700
-Wire Wire Line
-	6250 4500 6250 3700
-Connection ~ 4550 3600
-Connection ~ 6550 3400
-Wire Wire Line
-	6550 4500 6550 3400
-Connection ~ 5350 3200
-Wire Wire Line
-	5350 4500 5350 3200
-Wire Wire Line
-	7250 3800 7250 3100
-Wire Wire Line
-	4350 3800 4350 3100
-Wire Wire Line
-	7050 3100 7050 3600
-Wire Wire Line
-	7050 3600 4150 3600
-Wire Wire Line
-	4150 3600 4150 3100
-Wire Wire Line
-	6850 3100 6850 3400
-Wire Wire Line
-	6850 3400 3950 3400
-Wire Wire Line
-	6650 3100 6650 3200
-Wire Wire Line
-	6650 3200 3750 3200
-Wire Wire Line
-	3850 3100 3850 3300
-Wire Wire Line
-	3950 3400 3950 3100
-Wire Wire Line
-	3750 3200 3750 3100
-Wire Wire Line
-	3850 3300 6750 3300
-Wire Wire Line
-	6750 3300 6750 3100
-Wire Wire Line
-	4050 3100 4050 3500
-Wire Wire Line
-	4050 3500 6950 3500
-Wire Wire Line
-	6950 3500 6950 3100
-Wire Wire Line
-	4250 3100 4250 3700
-Wire Wire Line
-	4250 3700 7150 3700
-Wire Wire Line
-	7150 3700 7150 3100
-Wire Wire Line
-	4450 3100 4450 3900
-Wire Wire Line
-	4450 3900 7350 3900
-Wire Wire Line
-	7350 3900 7350 3100
-Wire Wire Line
-	5050 4500 5050 3300
-Connection ~ 5050 3300
-Connection ~ 4950 3500
-Wire Wire Line
-	4950 4500 4950 3500
-Connection ~ 4950 4100
-Connection ~ 5750 3900
-Wire Wire Line
-	5750 3900 5750 4400
-Wire Wire Line
-	5750 4400 6050 4400
-Wire Wire Line
-	6050 4400 6050 4500
-Connection ~ 5750 4100
-Wire Wire Line
-	4650 5400 4650 5300
-Wire Wire Line
-	7550 2300 7550 2400
 $Comp
 L GND #PWR01
@@
 F 0 "C2" H 6000 4200 50  0000 L CNN
 F 1 "220pF" H 6000 4000 50  0000 L CNN
-F 2 "" H 5950 4100 60  0001 C CNN
+F 2 "BSidesDFW_2018_Badge:C_Rect_L4.6mm_W2.0mm_P2.50mm_MKS02_FKP02" H 5950 4100 60  0001 C CNN
 F 3 "" H 5950 4100 60  0001 C CNN
 	1    5950 4100
@@
 F 0 "C1" H 4800 4200 50  0000 L CNN
 F 1 "220pF" H 4800 4000 50  0000 L CNN
-F 2 "" H 4750 4100 60  0001 C CNN
+F 2 "BSidesDFW_2018_Badge:C_Rect_L4.6mm_W2.0mm_P2.50mm_MKS02_FKP02" H 4750 4100 60  0001 C CNN
 F 3 "" H 4750 4100 60  0001 C CNN
 	1    4750 4100
@@
 F 0 "J2" H 7200 3150 60  0000 C CNN
 F 1 "RJ45" H 6850 3150 60  0000 C CNN
-F 2 "" H 7000 2650 60  0001 C CNN
+F 2 "BSidesDFW_2018_Badge:RJHSE538X" H 7000 2650 60  0001 C CNN
 F 3 "" H 7000 2650 60  0001 C CNN
 	1    7000 2650
@@
 F 0 "J4" H 6600 5450 60  0000 C CNN
 F 1 "RJ45" H 6250 5450 60  0000 C CNN
-F 2 "" H 6400 4950 60  0001 C CNN
+F 2 "BSidesDFW_2018_Badge:RJHSE538X" H 6400 4950 60  0001 C CNN
 F 3 "" H 6400 4950 60  0001 C CNN
 	1    6400 4950
@@
 F 0 "J3" H 5400 5450 60  0000 C CNN
 F 1 "RJ45" H 5050 5450 60  0000 C CNN
-F 2 "" H 5200 4950 60  0001 C CNN
+F 2 "BSidesDFW_2018_Badge:RJHSE538X" H 5200 4950 60  0001 C CNN
 F 3 "" H 5200 4950 60  0001 C CNN
 	1    5200 4950
@@
 F 0 "J1" H 4300 3150 60  0000 C CNN
 F 1 "RJ45" H 3950 3150 60  0000 C CNN
-F 2 "" H 4100 2650 60  0001 C CNN
+F 2 "BSidesDFW_2018_Badge:RJHSE538X" H 4100 2650 60  0001 C CNN
 F 3 "" H 4100 2650 60  0001 C CNN
 	1    4100 2650
@@
 Text Label 9650 6950 0    60   ~ 0
 Modified_by_altbier
+Wire Wire Line
+	4650 2300 4650 2400
+Wire Wire Line
+	5850 5300 5850 5400
+Connection ~ 6150 4100
+Wire Wire Line
+	6150 4500 6150 3800
+Wire Wire Line
+	7250 3800 4350 3800
+Connection ~ 6150 3800
+Connection ~ 4550 4100
+Wire Wire Line
+	4850 4500 4850 4400
+Wire Wire Line
+	4850 4400 4550 4400
+Wire Wire Line
+	4550 4400 4550 3600
+Connection ~ 6250 3700
+Wire Wire Line
+	6250 4500 6250 3700
+Connection ~ 4550 3600
+Connection ~ 6550 3400
+Wire Wire Line
+	6550 4500 6550 3400
+Connection ~ 5350 3200
+Wire Wire Line
+	5350 4500 5350 3200
+Wire Wire Line
+	7250 3800 7250 3100
+Wire Wire Line
+	4350 3800 4350 3100
+Wire Wire Line
+	7050 3100 7050 3600
+Wire Wire Line
+	7050 3600 4150 3600
+Wire Wire Line
+	4150 3600 4150 3100
+Wire Wire Line
+	6850 3100 6850 3400
+Wire Wire Line
+	6850 3400 3950 3400
+Wire Wire Line
+	6650 3100 6650 3200
+Wire Wire Line
+	6650 3200 3750 3200
+Wire Wire Line
+	3850 3100 3850 3300
+Wire Wire Line
+	3950 3400 3950 3100
+Wire Wire Line
+	3750 3200 3750 3100
+Wire Wire Line
+	3850 3300 6750 3300
+Wire Wire Line
+	6750 3300 6750 3100
+Wire Wire Line
+	4050 3100 4050 3500
+Wire Wire Line
+	4050 3500 6950 3500
+Wire Wire Line
+	6950 3500 6950 3100
+Wire Wire Line
+	4250 3100 4250 3700
+Wire Wire Line
+	4250 3700 7150 3700
+Wire Wire Line
+	7150 3700 7150 3100
+Wire Wire Line
+	4450 3100 4450 3900
+Wire Wire Line
+	4450 3900 7350 3900
+Wire Wire Line
+	7350 3900 7350 3100
+Wire Wire Line
+	5050 4500 5050 3300
+Connection ~ 5050 3300
+Connection ~ 4950 3500
+Wire Wire Line
+	4950 4500 4950 3500
+Connection ~ 4950 4100
+Connection ~ 5750 3900
+Wire Wire Line
+	5750 3900 5750 4400
+Wire Wire Line
+	5750 4400 6050 4400
+Wire Wire Line
+	6050 4400 6050 4500
+Connection ~ 5750 4100
+Wire Wire Line
+	4650 5400 4650 5300
+Wire Wire Line
+	7550 2300 7550 2400
+Wire Wire Line
+	4550 4100 4600 4100
+Wire Wire Line
+	4950 4100 4900 4100
+Wire Wire Line
+	5750 4100 5800 4100
+Wire Wire Line
+	6150 4100 6100 4100
 $EndSCHEMATC
